Commit message: Add: simulator lidar

File: src/gazebo_simulator_nodes/models/robot.xacro (robot description, xacro)
@@ -11,5 +11,5 @@
     <xacro:diff_drive/>
     <!-- <xacro:joint_state_publisher/> -->
-    <xacro:laser_frame/>
+    <xacro:lidar/>
     <xacro:ultrasonic/>
     <xacro:camera/>

File: src/gazebo_simulator_nodes/models/sensors.xacro (robot description, xacro)
@@ -1,8 +1,8 @@
 <?xml version="1.0"?>
 <robot xmlns:xacro="http://ros.org/wiki/xacro">
-    <xacro:macro name="laser_frame">
-        <xacro:cylinder_link name="laser_frame" mass="0.01" radius="0.01" length="0.005"/>
-        <xacro:fixed_joint name="laser_frame" child="laser_frame" origin_position="0 0 0.0425"/>
-        <gazebo reference="laser_frame">
+    <xacro:macro name="lidar">
+        <xacro:cylinder_link name="lidar" mass="0.01" radius="0.01" length="0.005"/>
+        <xacro:fixed_joint name="lidar" child="lidar" origin_position="0 0 0.0425"/>
+        <gazebo reference="lidar">
           <material>Gazebo/Red</material>
           <sensor name='gpu_lidar' type='gpu_lidar'>

Commit message: Add: imu for simulator

File: src/gazebo_simulator_nodes/models/robot.xacro (robot description, xacro)
@@ -9,4 +9,5 @@
     <xacro:fixed_joint name="base_footprint" parent="base_link" child="base_footprint"/>
     <xacro:box_link name="chassis" mass="2" x="${chassis_length}" y="${chassis_width}" z="${chassis_height}" material="black"/>
+    <xacro:imu/>
     <xacro:fixed_joint name="chassis" parent="base_link" child="chassis" origin_position="0 0 0.1"/>
     <xacro:diff_drive/>

File: src/gazebo_simulator_nodes/models/sensors.xacro (robot description, xacro)
@@ -125,3 +125,18 @@
     </gazebo>
 </xacro:macro>
+<xacro:macro name="imu">
+    <gazebo reference="chassis">
+      <sensor name="imu_sensor" type="imu">
+        <always_on>1</always_on>
+        <update_rate>20</update_rate>
+        <visualize>true</visualize>
+        <topic>simulator_imu</topic>
+      </sensor>
+    </gazebo>
+    <gazebo>
+      <plugin filename="libignition-gazebo-imu-system.so"
+        name="ignition::gazebo::systems::Imu">
+      </plugin>
+    </gazebo>
+</xacro:macro>
 </robot>
