Commit message: Huge polish, mostly just minor fixes, updated comments and some names, removed unused inports and other code, fixed indentation of xacro a sdf, added metadata, and other similar small stuff

File: src/gazebo_simulator_nodes/models/components.xacro (robot description, xacro)
@@ -1,4 +1,5 @@
 <?xml version="1.0"?>
 <robot xmlns:xacro="http://ros.org/wiki/xacro">
+<!-- basic building blocks -->
 <xacro:macro name="box_link" params="name mass x y z material:=red">
     <link name="${name}">
@@ -6,6 +7,6 @@
             <mass value="${mass}" />
             <inertia ixx="${(1/12) * mass * (y*y+z*z)}" ixy="0.0" ixz="0.0"
-                    iyy="${(1/12) * mass * (x*x+z*z)}" iyz="0.0"
-                    izz="${(1/12) * mass * (x*x+y*y)}" />
+                     iyy="${(1/12) * mass * (x*x+z*z)}" iyz="0.0"
+                     izz="${(1/12) * mass * (x*x+y*y)}" />
         </inertial>
         <visual>
@@ -23,10 +24,10 @@
 </xacro:macro>
 <xacro:macro name="cylinder_link" params="name mass radius length material:=red">
-  <link name="${name}">
+    <link name="${name}">
         <inertial>
             <mass value="${mass}" />
             <inertia ixx="${(1/12) * mass * (3*radius*radius + length*length)}" ixy="0.0" ixz="0.0"
-                    iyy="${(1/12) * mass * (3*radius*radius + length*length)}" iyz="0.0"
-                    izz="${(1/2) * mass * (radius*radius)}" />
+                     iyy="${(1/12) * mass * (3*radius*radius + length*length)}" iyz="0.0"
+                     izz="${(1/2) * mass * (radius*radius)}" />
         </inertial>
         <visual>
@@ -44,9 +45,9 @@
 </xacro:macro>
 <xacro:macro name="fixed_joint" params="name parent:=chassis child origin_position:='0 0 0' origin_orientation:='0 0 0'">
-  <joint name="${name}_joint" type="fixed">
-    <parent link="${parent}"/>
-    <child link="${child}"/>
-    <origin xyz="${origin_position}" rpy="${origin_orientation}"/>
-  </joint>
+    <joint name="${name}_joint" type="fixed">
+        <parent link="${parent}"/>
+        <child link="${child}"/>
+        <origin xyz="${origin_position}" rpy="${origin_orientation}"/>
+    </joint>
 </xacro:macro>
 <xacro:macro name="continuous_joint" params="name parent:=chassis child origin_position:='0 0 0' origin_orientation:='0 0 0' axis='0 0 0'">
@@ -58,4 +59,5 @@
     </joint>
 </xacro:macro>
+<!-- output components -->
 <xacro:macro name="diff_drive" params="">
     <xacro:cylinder_link name="left_front_wheel" mass="0.05" radius="${wheel_radius}" length="0.02" material="yellow"/>
@@ -68,89 +70,89 @@
     <xacro:continuous_joint name="right_rear_wheel" child="right_rear_wheel" origin_position="-0.05 -0.075 -0.025" origin_orientation="-1.5707 0 0" axis="0 0 1"/>
     <xacro:if value="$(arg use_sim)">
-      <ros2_control name="GazeboSimSystem" type="system">
-          <hardware>
-              <plugin>gz_ros2_control/GazeboSimSystem</plugin>
-          </hardware>
-          <joint name="left_front_wheel_joint">
-            <command_interface name="velocity">
-              <param name="min">-100</param>
-              <param name="max">100</param>
-            </command_interface>
-            <state_interface name="position"/>
-            <state_interface name="velocity"/>
-          </joint>
-          <joint name="right_front_wheel_joint">
-            <command_interface name="velocity">
-              <param name="min">-100</param>
-              <param name="max">100</param>
-            </command_interface>
-            <state_interface name="position"/>
-            <state_interface name="velocity"/>
-          </joint>
-          <joint name="left_rear_wheel_joint">
-              <command_interface name="velocity">
-                <param name="min">-100</param>
-                <param name="max">100</param>
-              </command_interface>
-              <state_interface name="position"/>
-              <state_interface name="velocity"/>
+        <ros2_control name="GazeboSimSystem" type="system">
+            <hardware>
+                <plugin>gz_ros2_control/GazeboSimSystem</plugin>
+            </hardware>
+            <joint name="left_front_wheel_joint">
+                <command_interface name="velocity">
+                    <param name="min">-100</param>
+                    <param name="max">100</param>
+                </command_interface>
+                <state_interface name="position"/>
+                <state_interface name="velocity"/>
             </joint>
-          <joint name="right_rear_wheel_joint">
-            <command_interface name="velocity">
-              <param name="min">-100</param>
-              <param name="max">100</param>
-            </command_interface>
-            <state_interface name="position"/>
-            <state_interface name="velocity"/>
-          </joint>
-      </ros2_control>
+            <joint name="right_front_wheel_joint">
+                <command_interface name="velocity">
+                    <param name="min">-100</param>
+                    <param name="max">100</param>
+                </command_interface>
+                <state_interface name="position"/>
+                <state_interface name="velocity"/>
+            </joint>
+            <joint name="left_rear_wheel_joint">
+                <command_interface name="velocity">
+                    <param name="min">-100</param>
+                    <param name="max">100</param>
+                </command_interface>
+                <state_interface name="position"/>
+                <state_interface name="velocity"/>
+            </joint>
+            <joint name="right_rear_wheel_joint">
+                <command_interface name="velocity">
+                    <param name="min">-100</param>
+                    <param name="max">100</param>
+                </command_interface>
+                <state_interface name="position"/>
+                <state_interface name="velocity"/>
+            </joint>
+        </ros2_control>
     </xacro:if>
     <xacro:unless value="$(arg use_sim)">
-      <ros2_control name="GazeboRealSystem" type="system">
-          <hardware>
-              <plugin>adeept_awr_diffdrive_control_plugin/AdeeptDiffDriveHardware</plugin>
-              <param name="motor_left_enable_pin">4</param>
-              <param name="motor_left_forward_pin">21</param>
-              <param name="motor_left_backward_pin">26</param>
-              <param name="motor_right_enable_pin">17</param>
-              <param name="motor_right_forward_pin">18</param>
-              <param name="motor_right_backward_pin">27</param>
-              <param name="max_motor_rotation_speed">18.0</param>
-          </hardware>
-          <joint name="left_front_wheel_joint">
-            <command_interface name="velocity">
-              <param name="min">-100</param>
-              <param name="max">100</param>
-            </command_interface>
-          </joint>
-          <joint name="right_front_wheel_joint">
-            <command_interface name="velocity">
-              <param name="min">-100</param>
-              <param name="max">100</param>
-            </command_interface>
-          </joint>
-          <joint name="left_rear_wheel_joint">
-              <command_interface name="velocity">
-                <param name="min">-100</param>
-                <param name="max">100</param>
-              </command_interface>
+        <ros2_control name="GazeboRealSystem" type="system">
+            <hardware>
+                <plugin>adeept_awr_diffdrive_control_plugin/AdeeptDiffDriveHardware</plugin>
+                <param name="motor_left_enable_pin">4</param>
+                <param name="motor_left_forward_pin">21</param>
+                <param name="motor_left_backward_pin">26</param>
+                <param name="motor_right_enable_pin">17</param>
+                <param name="motor_right_forward_pin">18</param>
+                <param name="motor_right_backward_pin">27</param>
+                <param name="max_motor_rotation_speed">18.0</param>
+            </hardware>
+            <joint name="left_front_wheel_joint">
+                <command_interface name="velocity">
+                    <param name="min">-100</param>
+                    <param name="max">100</param>
+                </command_interface>
             </joint>
-          <joint name="right_rear_wheel_joint">
-              <command_interface name="velocity">
-                <param name="min">-100</param>
-                <param name="max">100</param>
-              </command_interface>
+            <joint name="right_front_wheel_joint">
+                <command_interface name="velocity">
+                    <param name="min">-100</param>
+                    <param name="max">100</param>
+                </command_interface>
+            </joint>
+            <joint name="left_rear_wheel_joint">
+                <command_interface name="velocity">
+                    <param name="min">-100</param>
+                    <param name="max">100</param>
+                </command_interface>
+                </joint>
+            <joint name="right_rear_wheel_joint">
+                <command_interface name="velocity">
+                    <param name="min">-100</param>
+                    <param name="max">100</param>
+                </command_interface>
             </joint>
         </ros2_control>
     </xacro:unless>
     <gazebo>
-      <plugin filename="/opt/ros/iron/lib/libgz_ros2_control-system.so" name="gz_ros2_control::GazeboSimROS2ControlPlugin">
-        <parameters>$(find adeept_awr_diffdrive_control_plugin)/config/controllers.yaml</parameters>
-        <parameters>$(find adeept_awr_diffdrive_control_plugin)/config/controllers_sim.yaml</parameters>
-        <ros>
-          <remapping>/diff_drive_controller/cmd_vel_unstamped:=/cmd_vel</remapping>
-          <remapping>/robot_description:=/controller_manager/robot_description</remapping>
-        </ros>
-      </plugin>
+        <plugin filename="/opt/ros/iron/lib/libgz_ros2_control-system.so" name="gz_ros2_control::GazeboSimROS2ControlPlugin">
+            <parameters>$(find adeept_awr_diffdrive_control_plugin)/config/controllers.yaml</parameters>
+            <parameters>$(find adeept_awr_diffdrive_control_plugin)/config/controllers_sim.yaml</parameters>
+            <ros>
+                <remapping>/diff_drive_controller/cmd_vel_unstamped:=/cmd_vel</remapping>
+                <remapping>/robot_description:=/controller_manager/robot_description</remapping>
+            </ros>
+        </plugin>
     </gazebo>
 </xacro:macro>
@@ -171,11 +173,3 @@
     </gazebo>
 </xacro:macro>
-<xacro:macro name="joint_state_publisher">
-    <gazebo>
-        <plugin name="ignition::gazebo::systems::JointStatePublisher" filename="libignition-gazebo-joint-state-publisher-system.so">
-            <update_rate>10</update_rate>
-            <topic>joint_states</topic>
-        </plugin>
-    </gazebo>
-</xacro:macro>
 </robot>

File: src/gazebo_simulator_nodes/models/robot.xacro (robot description, xacro)
@@ -5,4 +5,5 @@
     <xacro:include filename="components.xacro"/>
     <xacro:include filename="sensors.xacro"/>
+    <!-- robot -->
     <link name="base_link"/>
     <link name="base_footprint"/>
@@ -12,5 +13,4 @@
     <xacro:fixed_joint name="chassis" parent="base_link" child="chassis" origin_position="0 0 0.1"/>
     <xacro:diff_drive/>
-    <xacro:joint_state_publisher/>
     <xacro:lidar/>
     <xacro:ultrasonic/>

File: src/gazebo_simulator_nodes/models/sensors.xacro (robot description, xacro)
@@ -1,77 +1,77 @@
 <?xml version="1.0"?>
 <robot xmlns:xacro="http://ros.org/wiki/xacro">
-    <xacro:macro name="lidar">
-        <xacro:cylinder_link name="lidar" mass="0.01" radius="0.025" length="0.02"/>
-        <xacro:fixed_joint name="lidar" child="lidar" origin_position="0 0 0.05"/>
-        <gazebo reference="lidar">
-          <sensor name='gpu_lidar' type='gpu_lidar'>
+<xacro:macro name="lidar">
+    <xacro:cylinder_link name="lidar" mass="0.01" radius="0.025" length="0.02"/>
+    <xacro:fixed_joint name="lidar" child="lidar" origin_position="0 0 0.05"/>
+    <gazebo reference="lidar">
+        <sensor name='gpu_lidar' type='gpu_lidar'>
             <topic>simulator_lidar</topic>
             <update_rate>20</update_rate>
             <lidar>
-              <scan>
-                <horizontal>
-                  <samples>360</samples>
-                  <resolution>1</resolution>
-                  <min_angle>-3.14</min_angle>
-                  <max_angle>3.14</max_angle>
-                </horizontal>
-                <vertical>
-                  <samples>1</samples>
-                  <resolution>1</resolution>
-                  <min_angle>0</min_angle>
-                  <max_angle>0</max_angle>
-                </vertical>
-              </scan>
-              <range>
-                <min>0.08</min>
-                <max>10</max>
-                <resolution>0.01</resolution>
-              </range>
-              <noise>
-                <type>none</type>
-                <mean>0</mean>
-                <stddev>0</stddev>
-              </noise>
-              <visibility_mask>4294967295</visibility_mask>
+                <scan>
+                    <horizontal>
+                        <samples>360</samples>
+                        <resolution>1</resolution>
+                        <min_angle>-3.14</min_angle>
+                        <max_angle>3.14</max_angle>
+                    </horizontal>
+                    <vertical>
+                        <samples>1</samples>
+                        <resolution>1</resolution>
+                        <min_angle>0</min_angle>
+                        <max_angle>0</max_angle>
+                    </vertical>
+                </scan>
+                <range>
+                    <min>0.08</min>
+                    <max>10</max>
+                    <resolution>0.01</resolution>
+                </range>
+                <noise>
+                    <type>none</type>
+                    <mean>0</mean>
+                    <stddev>0</stddev>
+                </noise>
+                <visibility_mask>4294967295</visibility_mask>
             </lidar>
-          </sensor>
-      </gazebo>
+        </sensor>
+    </gazebo>
 </xacro:macro>
 <xacro:macro name="ultrasonic">
-  <xacro:box_link name="ultrasonic" mass="0.01" x="0.01" y="0.03" z="0.015" material="blue"/>
-  <xacro:fixed_joint name="ultrasonic" child="ultrasonic" origin_position="0.065 0 -0.02"/>
-  <gazebo reference="ultrasonic">
-    <sensor name='gpu_lidar_ultra' type='gpu_lidar'>
-      <topic>simulator_ultrasonic</topic>
-      <update_rate>20</update_rate>
-      <lidar>
-        <scan>
-          <horizontal>
-            <samples>3</samples>
-            <resolution>1</resolution>
-            <min_angle>-0.1308</min_angle>
-            <max_angle>0.1308</max_angle>
-          </horizontal>
-          <vertical>
-            <samples>1</samples>
-            <resolution>1</resolution>
-            <min_angle>0</min_angle>
-            <max_angle>0</max_angle>
-          </vertical>
-        </scan>
-        <range>
-          <min>0.02</min>
-          <max>4</max>
-          <resolution>0.01</resolution>
-        </range>
-        <noise>
-          <type>none</type>
-          <mean>0</mean>
-          <stddev>0</stddev>
-        </noise>
-        <visibility_mask>4294967295</visibility_mask>
-      </lidar>
-    </sensor>
-  </gazebo>
+    <xacro:box_link name="ultrasonic" mass="0.01" x="0.01" y="0.03" z="0.015" material="blue"/>
+    <xacro:fixed_joint name="ultrasonic" child="ultrasonic" origin_position="0.065 0 -0.02"/>
+    <gazebo reference="ultrasonic">
+        <sensor name='gpu_lidar_ultra' type='gpu_lidar'>
+            <topic>simulator_ultrasonic</topic>
+            <update_rate>20</update_rate>
+            <lidar>
+                <scan>
+                    <horizontal>
+                        <samples>3</samples>
+                        <resolution>1</resolution>
+                        <min_angle>-0.1308</min_angle>
+                        <max_angle>0.1308</max_angle>
+                    </horizontal>
+                    <vertical>
+                        <samples>1</samples>
+                        <resolution>1</resolution>
+                        <min_angle>0</min_angle>
+                        <max_angle>0</max_angle>
+                    </vertical>
+                </scan>
+                <range>
+                    <min>0.02</min>
+                    <max>4</max>
+                    <resolution>0.01</resolution>
+                </range>
+                <noise>
+                    <type>none</type>
+                    <mean>0</mean>
+                    <stddev>0</stddev>
+                </noise>
+                <visibility_mask>4294967295</visibility_mask>
+            </lidar>
+        </sensor>
+    </gazebo>
 </xacro:macro>
 <xacro:macro name="camera">
@@ -81,5 +81,5 @@
             <topic>simulator_camera</topic>
             <update_rate>30</update_rate>
-            <camera name='__default__'>
+            <camera>
                 <horizontal_fov>1.0469999999999999</horizontal_fov>
                 <image>
@@ -108,7 +108,7 @@
     <gazebo reference="line_tracking_${suffix}">
         <sensor name='line_tracking_${suffix}' type='camera'>
-            <topic>line_tracking</topic>
+            <topic>simulator_line_visibility</topic>
             <update_rate>10</update_rate>
-            <camera name='__default__'>
+            <camera>
                 <horizontal_fov>0.11</horizontal_fov>
                 <image>
